File: ampli.kicad_pcb (KiCad board)
At the start: 2 copper layers, 110 x 100 mm, 51 parts, among them J2 Conn_01x02, J3 Conn_01x03, Q1 2N2907, Q10 TIP32, Q11 BD138, Q12 TIP31, Q13 2N2222, Q2 2N2907, Q3 2N2907, Q4 2N2222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

Commit message: .
Parts:
- U2: moved to F.Cu
- moved R11 72.2 mm to (136.3, 77.2), turned to 90 degrees
- moved HS1 60.5 mm to (125.3, 74.2), turned to -90 degrees
- moved Q10 58.8 mm to (127.7, 76.7)
- moved C4 48.1 mm to (67.2, 44.5)
- moved C6 47.2 mm to (79.6, 44.7)
- moved R13 45.5 mm to (113.0, 85.6), turned to -90 degrees
- moved Q9 44.9 mm to (114.9, 71.8), turned to -90 degrees
- moved C8 43.3 mm to (125.1, 45.5), turned to -90 degrees
- moved U1 43.1 mm to (91.3, 48.3), turned to 0 degrees
- moved C5 40.1 mm to (67.3, 54.9)
- moved C7 38.5 mm to (79.7, 54.6)
- moved Dz1 38.4 mm to (66.9, 69.5), turned to -90 degrees
- moved C11 36.9 mm to (169.0, 52.2), turned to 180 degrees
- moved R8 36.2 mm to (164.5, 113.2), turned to 180 degrees
- moved C9 35.8 mm to (115.2, 66.9), turned to 90 degrees
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Connections:
- Q12 pad 1: Net-(Q11-Pad1) -> Net-(Q11-Pad2)
- Q12 pad 2: Net-(Q11-Pad2) -> Net-(Q11-Pad1)
- R12 pad 2: Net-(Q11-Pad2) -> Net-(Q11-Pad1)
Routing:
- net +12V: track 312.9 -> 0.00 mm, vias 1 -> 0
- net -12V: track 212.9 -> 0.00 mm
- net Net-(R11-Pad2): track 116.1 -> 0.00 mm
- net Net-(Q6-Pad3): track 110.6 -> 0.00 mm, vias 1 -> 0
- net Net-(C2-Pad1): track 89.4 -> 0.57 mm
- net Net-(Q10-Pad2): track 58.9 -> 0.00 mm
- net Net-(Q11-Pad2): track 40.0 -> 0.00 mm
- net Net-(C2-Pad2): track 39.9 -> 0.42 mm
- net Net-(Q2-Pad2): track 39.3 -> 0.00 mm
- net Net-(Q11-Pad1): track 33.1 -> 0.00 mm
- net /HP: track 32.3 -> 0.00 mm
- net Net-(C1-Pad1): track 26.5 -> 0.00 mm
- net Net-(Q6-Pad2): track 26.1 -> 0.00 mm
- net Net-(Dz1-Pad2): track 25.5 -> 0.89 mm
- net Net-(Q3-Pad1): track 22.6 -> 0.00 mm
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- removed copper zone on B.Cu, net GND
- removed copper zone on F.Cu, net GND

Commit message: .
Parts:
- C1, C4, C6: footprint Capacitor_THT:CP_Radial_D8.0mm_P5.00mm -> CmpAmpliAudioTR:CP_Radial_D8.0mm_P5.00mm
- C10, C3, C8: footprint Capacitor_THT:CP_Radial_D12.5mm_P5.00mm -> CmpAmpliAudioTR:CP_Radial_D12.5mm_P5.00mm
- C11, C2, C5, C7, C9: footprint Capacitor_THT:C_Rect_L7.2mm_W3.5mm_P5.00mm_FKS2_FKP2_MKS2_MKP2 -> CmpAmpliAudioTR:C_Rect_L7.2mm_W3.5mm_P5.00mm_FKS2_FKP2_MKS2_MKP2
- D1: footprint Diode_THT:D_DO-35_SOD27_P7.62mm_Horizontal -> CmpAmpliAudioTR:D_DO-35_SOD27_P10.16mm_Horizontal
- D2, Dz1: footprint Diode_THT:D_DO-35_SOD27_P10.16mm_Horizontal -> CmpAmpliAudioTR:D_DO-35_SOD27_P10.16mm_Horizontal
- HS1, HS2: footprint Heatsink:Heatsink_Fischer_SK104-STC-STIC_35x13mm_2xDrill2.5mm -> CmpAmpliAudioTR:Heatsink_Fischer_SK104-STC-STIC_35x13mm_2xDrill2.5mm
- J2: footprint Connector_Phoenix_MSTB:PhoenixContact_MSTBVA_2,5_2-G-5,08_1x02_P5.08mm_Vertical -> CmpAmpliAudioTR:PhoenixContact_MSTBVA_2,5_2-G-5,08_1x02_P5.08mm_Vertical
- J3: footprint Connector_Phoenix_MSTB:PhoenixContact_MSTBVA_2,5_3-G-5,08_1x03_P5.08mm_Vertical -> CmpAmpliAudioTR:PhoenixContact_MSTBVA_2,5_3-G-5,08_1x03_P5.08mm_Vertical
- Q1, Q13, Q2, Q3, Q4, Q5, Q6, Q7: footprint Package_TO_SOT_THT:TO-18-3 -> CmpAmpliAudioTR:TO-18-3
- Q10, Q12: footprint Package_TO_SOT_THT:TO-220-3_Vertical -> CmpAmpliAudioTR:TO-220-3_Vertical
- Q11, Q8, Q9: footprint Package_TO_SOT_THT:TO-126-3_Vertical -> CmpAmpliAudioTR:TO-126-3_Vertical
- R1, R10, R13, R14, R15, R16, R2, R3, R4, R5, R6, R7, R8, R9: footprint Resistor_THT:R_Axial_DIN0207_L6.3mm_D2.5mm_P10.16mm_Horizontal -> CmpAmpliAudioTR:R_Axial_DIN0207_L6.3mm_D2.5mm_P10.16mm_Horizontal
- RV1, RV2: footprint Potentiometer_THT:Potentiometer_Bourns_3296W_Vertical -> CmpAmpliAudioTR:Potentiometer_Bourns_3296W_Vertical
- moved D1 2.29 mm to (110.5, 29.1)
Routing:
- net Net-(C2-Pad1): track 0.57 -> 0.00 mm

Commit message: .
Parts:
- moved U2 0.32 mm to (92.1, 125.0)
Routing:
- net +12V: track 0.00 -> 230.4 mm
- net -12V: track 0.00 -> 201.3 mm
- net Net-(C2-Pad1): track 0.00 -> 127.5 mm
- net Net-(R11-Pad2): track 0.00 -> 105.9 mm
- net Net-(Q6-Pad3): track 0.00 -> 72.3 mm
- net Net-(Q6-Pad2): track 0.00 -> 45.4 mm
- net Net-(C2-Pad2): track 0.42 -> 41.6 mm
- net Net-(Q11-Pad1): track 0.00 -> 40.7 mm
- net Net-(Q1-Pad1): track 0.00 -> 36.0 mm
- net Net-(C1-Pad2): track 0.00 -> 34.3 mm
- net Net-(C1-Pad1): track 0.00 -> 25.2 mm
- net Net-(Q10-Pad2): track 0.00 -> 23.6 mm
- net Net-(Q8-Pad3): track 0.00 -> 23.4 mm
- net Net-(C3-Pad1): track 0.00 -> 21.5 mm
- net Net-(Q2-Pad2): track 0.00 -> 18.5 mm
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- added copper zone on B.Cu, net GND
- added copper zone on F.Cu, net GND

Commit message: .
Parts:
- moved R12 3.56 mm to (145.0, 93.0)
- moved D1 3.43 mm to (107.1, 29.0)
Routing:
- net Net-(R11-Pad2): track 105.9 -> 86.0 mm, vias 0 -> 2
- net (no net): track 0.00 -> 16.1 mm, vias 4 -> 6
- net Net-(Q11-Pad1): track 40.7 -> 35.4 mm
- net Net-(Q6-Pad3): track 72.3 -> 67.1 mm, vias 0 -> 2
- net -12V: track 201.3 -> 201.1 mm, vias 0 -> 2

Commit message: .
Parts:
- moved Q10 2.03 mm to (129.7, 76.7)
- moved Q12 1.87 mm to (159.6, 75.7)
Routing:
- net Net-(R11-Pad2): track 86.0 -> 90.3 mm
- net +12V: track 230.6 -> 234.0 mm
- net Net-(Q10-Pad1): track 13.7 -> 15.8 mm
- net Net-(C2-Pad1): track 127.5 -> 129.3 mm
- net Net-(Q11-Pad1): track 35.4 -> 37.1 mm
- net Net-(Q11-Pad2): track 10.7 -> 9.01 mm
- net Net-(Q6-Pad3): track 67.1 -> 66.3 mm
- net (no net): track 16.1 -> 15.6 mm
Other:
- board text added: "MARCEAU Jérémy Amplificateur Audio"

Commit message: .
Routing:
- net Net-(Q11-Pad1): track 37.1 -> 40.8 mm
Changed lines of the file:
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@@
   (segment (start 76.638724 79.317276) (end 76.638724 74.987724) (width 0.6) (layer "B.Cu") (net 11))
   (segment (start 68.707 81.407) (end 66.929 79.629) (width 0.6) (layer "B.Cu") (net 11))
+  (segment (start 143.489 31.1585) (end 145.376276 33.045776) (width 0.6) (layer "B.Cu") (net 12))
   (segment (start 131.5585 31.1585) (end 143.489 31.1585) (width 1.2) (layer "B.Cu") (net 12))
-  (segment (start 143.489 31.1585) (end 145.376276 33.045776) (width 0.6) (layer "B.Cu") (net 12))
   (segment (start 85.344 84.328) (end 86.063724 85.047724) (width 0.6) (layer "B.Cu") (net 13))
   (segment (start 87.941724 102.319724) (end 87.941724 85.301724) (width 0.6) (layer "B.Cu") (net 13))
@@
   (segment (start 153.797 97.663) (end 156.21 95.25) (width 0.6) (layer "B.Cu") (net 23))
   (segment (start 166.624 95.758) (end 166.624 100.33) (width 0.6) (layer "B.Cu") (net 23))
-  (segment (start 133.257302 74.168) (end 129.723 74.168) (width 0.6) (layer "B.Cu") (net 24))
+  (segment (start 133.257302 74.168) (end 129.723 74.168) (width 1.2) (layer "B.Cu") (net 24))
   (segment (start 121.666 74.168) (end 119.293 71.795) (width 0.6) (layer "B.Cu") (net 24))
   (segment (start 114.941 71.795) (end 119.293 71.795) (width 0.6) (layer "B.Cu") (net 24))
-  (segment (start 136.271 77.181698) (end 133.257302 74.168) (width 0.6) (layer "B.Cu") (net 24))
+  (segment (start 136.271 77.181698) (end 133.257302 74.168) (width 1.2) (layer "B.Cu") (net 24))
   (segment (start 129.723 74.168) (end 121.666 74.168) (width 0.6) (layer "B.Cu") (net 24))
   (segment (start 118.832 74.335) (end 121.205 76.708) (width 0.6) (layer "B.Cu") (net 25))
@@
   (segment (start 114.941 74.335) (end 118.832 74.335) (width 0.6) (layer "B.Cu") (net 25))
   (segment (start 161.919 79.502) (end 156.083 79.502) (width 0.6) (layer "B.Cu") (net 26))
-  (segment (start 156.083 72.644) (end 156.591 72.644) (width 0.6) (layer "B.Cu") (net 26))
   (segment (start 145.034 72.644) (end 145.669 73.279) (width 0.6) (layer "B.Cu") (net 26))
-  (segment (start 145.034 72.644) (end 156.591 72.644) (width 0.6) (layer "B.Cu") (net 26))
   (segment (start 158.877 72.644) (end 159.385 73.152) (width 0.6) (layer "B.Cu") (net 26))
-  (segment (start 154.305 74.422) (end 156.083 72.644) (width 0.6) (layer "B.Cu") (net 26))
+  (segment (start 159.06 72.644) (end 159.568 73.152) (width 1.2) (layer "B.Cu") (net 26))
   (segment (start 166.872 74.549) (end 161.919 79.502) (width 0.6) (layer "B.Cu") (net 26))
   (segment (start 156.083 79.502) (end 154.305 77.724) (width 0.6) (layer "B.Cu") (net 26))
+  (segment (start 145.034 72.644) (end 159.06 72.644) (width 1.2) (layer "B.Cu") (net 26))
+  (segment (start 155.575 73.152) (end 159.568 73.152) (width 0.6) (layer "B.Cu") (net 26))
   (segment (start 154.305 77.724) (end 154.305 74.422) (width 0.6) (layer "B.Cu") (net 26))
-  (segment (start 156.591 72.644) (end 158.877 72.644) (width 0.6) (layer "B.Cu") (net 26))
+  (segment (start 154.305 74.422) (end 155.575 73.152) (width 0.6) (layer "B.Cu") (net 26))
   (segment (start 162.052 110.744) (end 164.465 113.157) (width 0.6) (layer "B.Cu") (net 27))
   (segment (start 162.052 103.495) (end 162.052 110.744) (width 0.6) (layer "B.Cu") (net 27))
